Commit message: add lidar_link and geometry

File: rover_roahm_description/urdf/rover_roahm.urdf.xacro (robot description, xacro)
@@ -95,4 +95,7 @@
     <color rgba="0 0 0 1"/>
   </material>
+  <material name="lidar_mat">
+    <color rgba="0.8 0.6 0 1"/>
+  </material>
   <!-- Null inertial element. This is needed to make the model work with
        Gazebo. -->
@@ -346,44 +349,71 @@
     	<material>Gazebo/Green</material>
   	</gazebo>
-   <joint name="left_eye_to_head" type="fixed">
-    <parent link="eye_link"/>
-    <child link="left_eye"/>
-    <origin xyz="0.03 0.03 0.0" rpy="0.0 0.0 0.0"/>
-   </joint>
-   <joint name="right_eye_to_head" type="fixed">
-    <parent link="eye_link"/>
-    <child link="right_eye"/>
-    <origin xyz="0.03 -0.03 0.0" rpy="0.0 0.0 0.0"/>
-   </joint>
-   <joint name="base_link_to_eye" type="fixed">
+  <joint name="left_eye_to_head" type="fixed">
+  <parent link="eye_link"/>
+  <child link="left_eye"/>
+  <origin xyz="0.03 0.03 0.0" rpy="0.0 0.0 0.0"/>
+  </joint>
+  <joint name="right_eye_to_head" type="fixed">
+  <parent link="eye_link"/>
+  <child link="right_eye"/>
+  <origin xyz="0.03 -0.03 0.0" rpy="0.0 0.0 0.0"/>
+  </joint>
+  <joint name="base_link_to_eye" type="fixed">
+  <parent link="base_link"/>
+  <child link="eye_link"/>
+  <origin xyz="${chassis_length /2 + 0.03} 0.0 0.22" rpy="0.0 0.0 0.0"/>
+  </joint>
+  <joint name="imu_joint" type="fixed">
+  <axis xyz="1 0 0"/>
+  <origin xyz="0.06 -0.054 0.16" rpy="3.1416 0 0"/>
+  <parent link="base_link"/>
+  <child link="imu_link"/>
+  </joint>
+  <link name="imu_link">
+    <inertial>
+      <mass value="0.001"/>
+      <origin rpy="0 0 0" xyz="0 0 0"/>
+      <inertia ixx="0.0001" ixy="0" ixz="0" iyy="0.000001" iyz="0" izz="0.0001"/>
+    </inertial>
+    <visual>
+      <origin rpy="0 0 0" xyz="0 0 0"/>
+      <geometry>
+        <box size="0.1 0.1 0.005"/>
+      </geometry>
+      <material name="chassis_mat"/>
+    </visual>
+    <collision>
+      <origin rpy="0 0 0" xyz="0 0 0"/>
+      <geometry>
+        <box size=".001 .001 .001"/>
+      </geometry>
+    </collision>
+  </link>
+  <joint name="lidar_joint" type="fixed">
+    <axis xyz="1 0 0"/>
+    <origin xyz="0.19 0 0.12" rpy="0 0 0"/>
     <parent link="base_link"/>
-    <child link="eye_link"/>
-    <origin xyz="${chassis_length /2 + 0.03} 0.0 0.1" rpy="0.0 0.0 0.0"/>
-   </joint>
-    <joint name="imu_joint" type="fixed">
-		<axis xyz="1 0 0"/>
-		<origin xyz="0.06 -0.054 0.16" rpy="3.1416 0 0"/>
-		<parent link="base_link"/>
-		<child link="imu_link"/>
-	</joint>
-	<link name="imu_link">
-	  <inertial>
-	    <mass value="0.001"/>
-	    <origin rpy="0 0 0" xyz="0 0 0"/>
-	    <inertia ixx="0.0001" ixy="0" ixz="0" iyy="0.000001" iyz="0" izz="0.0001"/>
-	  </inertial>
-	  <visual>
-	    <origin rpy="0 0 0" xyz="0 0 0"/>
-	    <geometry>
-	      <box size="0.001 0.001 0.001"/>
-	    </geometry>
-	  </visual>
-	  <collision>
-	    <origin rpy="0 0 0" xyz="0 0 0"/>
-	    <geometry>
-	      <box size=".001 .001 .001"/>
-	    </geometry>
-	  </collision>
-	</link>
+    <child link="lidar_link"/>
+  </joint>
+  <link name="lidar_link">
+    <inertial>
+      <mass value="0.001"/>
+      <origin rpy="0 0 0" xyz="0 0 0"/>
+      <inertia ixx="0.0001" ixy="0" ixz="0" iyy="0.000001" iyz="0" izz="0.0001"/>
+    </inertial>
+    <visual>
+      <origin rpy="0 0 0" xyz="0 0 0"/>
+      <geometry>
+        <cylinder length="0.07" radius="0.025"/>
+      </geometry>
+      <material name="lidar_mat"/>
+    </visual>
+    <collision>
+      <origin rpy="0 0 0" xyz="0 0 0"/>
+      <geometry>
+        <box size=".001 .001 .001"/>
+      </geometry>
+    </collision>
+  </link>
   <!-- Chassis -->
   <link name="chassis">

Commit message: change imu_link name to imu

File: rover_roahm_description/urdf/rover_roahm.urdf.xacro (robot description, xacro)
@@ -368,7 +368,7 @@
   <origin xyz="0.06 -0.054 0.16" rpy="3.1416 0 0"/>
   <parent link="base_link"/>
-  <child link="imu_link"/>
-  </joint>
-  <link name="imu_link">
+  <child link="imu"/>
+  </joint>
+  <link name="imu">
     <inertial>
       <mass value="0.001"/>
